File: Cryptuino01_MOV.sch (KiCad schematic (older format))
At the start: 30 parts, among them J1 USB_C_Receptacle_USB2.0, J2 Conn_01x06_Female, J3 Conn_01x08_Female, U1 FT245RL, U2 74HC02, U3 74HC00, U4 ATtiny4313-MU

Commit message: done_nice_now
Parts:
- C1, C2, C3, C4, C5, C6, C7: footprint Resistor_SMD:R_0805_2012Metric -> Capacitor_SMD:C_0805_2012Metric
- F1: footprint Resistor_SMD:R_0805_2012Metric -> Fuse:Fuse_0805_2012Metric
- L1: footprint Resistor_SMD:R_0805_2012Metric -> Inductor_SMD:L_0805_2012Metric
Changed lines of the file:
@@
 F 0 "F1" V 2110 4300 50  0000 C CNN
 F 1 "Polyfuse_300mA" H 1886 4300 50  0000 C CNN
-F 2 "Resistor_SMD:R_0805_2012Metric" H 2050 4100 50  0001 L CNN
+F 2 "Fuse:Fuse_0805_2012Metric" H 2050 4100 50  0001 L CNN
 F 3 "~" H 2000 4300 50  0001 C CNN
 	1    2000 4300
@@
 F 0 "L1" V 2656 4300 50  0000 C CNN
 F 1 "1mH" V 2485 4300 50  0000 C CNN
-F 2 "Resistor_SMD:R_0805_2012Metric" H 2550 4300 50  0001 C CNN
+F 2 "Inductor_SMD:L_0805_2012Metric" H 2550 4300 50  0001 C CNN
 F 3 "~" H 2550 4300 50  0001 C CNN
 	1    2550 4300
@@
 F 0 "C3" H 3292 4496 50  0000 L CNN
 F 1 "10uF" H 3292 4405 50  0000 L CNN
-F 2 "Resistor_SMD:R_0805_2012Metric" H 3200 4450 50  0001 C CNN
+F 2 "Capacitor_SMD:C_0805_2012Metric" H 3200 4450 50  0001 C CNN
 F 3 "~" H 3200 4450 50  0001 C CNN
 	1    3200 4450
@@
 F 0 "C4" H 8742 5946 50  0000 L CNN
 F 1 "100nF" H 8742 5855 50  0000 L CNN
-F 2 "Resistor_SMD:R_0805_2012Metric" H 8650 5900 50  0001 C CNN
+F 2 "Capacitor_SMD:C_0805_2012Metric" H 8650 5900 50  0001 C CNN
 F 3 "~" H 8650 5900 50  0001 C CNN
 	1    8650 5900
@@
 F 0 "C5" H 9292 5946 50  0000 L CNN
 F 1 "100nF" H 9292 5855 50  0000 L CNN
-F 2 "Resistor_SMD:R_0805_2012Metric" H 9200 5900 50  0001 C CNN
+F 2 "Capacitor_SMD:C_0805_2012Metric" H 9200 5900 50  0001 C CNN
 F 3 "~" H 9200 5900 50  0001 C CNN
 	1    9200 5900
@@
 F 0 "C6" H 10392 5946 50  0000 L CNN
 F 1 "100nF" H 10392 5855 50  0000 L CNN
-F 2 "Resistor_SMD:R_0805_2012Metric" H 10300 5900 50  0001 C CNN
+F 2 "Capacitor_SMD:C_0805_2012Metric" H 10300 5900 50  0001 C CNN
 F 3 "~" H 10300 5900 50  0001 C CNN
 	1    10300 5900
@@
 F 0 "C7" H 10892 5946 50  0000 L CNN
 F 1 "10uF" H 10892 5855 50  0000 L CNN
-F 2 "Resistor_SMD:R_0805_2012Metric" H 10800 5900 50  0001 C CNN
+F 2 "Capacitor_SMD:C_0805_2012Metric" H 10800 5900 50  0001 C CNN
 F 3 "~" H 10800 5900 50  0001 C CNN
 	1    10800 5900
@@
 F 0 "C2" H 3133 4404 50  0000 R CNN
 F 1 "100nF" H 3252 4495 50  0000 R CNN
-F 2 "Resistor_SMD:R_0805_2012Metric" H 2950 4450 50  0001 C CNN
+F 2 "Capacitor_SMD:C_0805_2012Metric" H 2950 4450 50  0001 C CNN
 F 3 "~" H 2950 4450 50  0001 C CNN
 	1    2950 4450
@@
 F 0 "C1" H 1183 1154 50  0000 R CNN
 F 1 "100nF" H 1302 1245 50  0000 R CNN
-F 2 "Resistor_SMD:R_0805_2012Metric" H 1000 1200 50  0001 C CNN
+F 2 "Capacitor_SMD:C_0805_2012Metric" H 1000 1200 50  0001 C CNN
 F 3 "~" H 1000 1200 50  0001 C CNN
 	1    1000 1200
